File: pcb/modelh.kicad_pcb (KiCad board)
At the start: 2 copper layers, 150 x 38 mm, 51 parts, among them J1 USB_B, J2 Conn_cols, J3 Conn_rows, J4 Conn_leds, J5 Conn_02x03_Odd_Even, J6 Conn_02x05_Odd_Even, J7 Conn_01x05, J8 Conn_01x05, J9 Conn_01x05, SW1 SW_Push, U1 STM32F103C8Tx, U2 AMS1117-3.3, Y1 8MHz

Commit message: Upgrading to modern Kicad
Other:
- net class Default removed
